File: Boards/main_plate.brd (EAGLE design)
At the start: 89 x 63 mm, 18 parts, among them IC1 ULN2003AN

Commit message: add nodeMCU code
Parts:
- added JP8: (no value), pinhead:1X01
Connections:
- net +5V: now also JP8.1
Routing:
- net +5V: track 57.2 -> 59.8 mm
Changed lines of the file:
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@@
 </layers>
 <board>
-<fusionsync huburn="a.cGVyc29uYWw6dWUyZGM4MWM3" projecturn="a.cGVyc29uYWw6dWUyZGM4MWM3I0QyMDE4MDQxMzEyNzQyMzUyNg" f3durn="urn:adsk.wipprod:dm.lineage:yT0FvSQqTkuGDmDyUKnVDQ" pcbguid="6065538a-f9ac-4097-be1e-d1dee08dff7d" lastpulledtime="" lastsyncedchangeguid="b757bd44-08c8-8315-7388-945c0c851f30"/>
+<fusionsync huburn="a.cGVyc29uYWw6dWUyZGM4MWM3" projecturn="a.cGVyc29uYWw6dWUyZGM4MWM3I0QyMDE4MDQxMzEyNzQyMzUyNg" f3durn="urn:adsk.wipprod:dm.lineage:yT0FvSQqTkuGDmDyUKnVDQ" pcbguid="6065538a-f9ac-4097-be1e-d1dee08dff7d" lastpulledtime="" lastsyncedchangeguid="c7acfe65-8adb-827d-d36e-46d70be79035"/>
 <plain>
 <wire x1="14" y1="0" x2="77" y2="0" width="0" layer="20"/>
@@
 <attribute name="OC_NEWARK" value="unknown" x="6.35" y="44.45" size="1.778" layer="27" rot="R270" display="off"/>
 </element>
+<element name="JP8" library="pinhead" library_urn="urn:adsk.eagle:library:325" package="1X01" package3d_urn="urn:adsk.eagle:package:22485/2" value="" x="57.15" y="8.89"/>
 </elements>
 <signals>
@@
 <wire x1="69.5" y1="9.24" x2="64.44" y2="4.18" width="1.016" layer="16"/>
 <wire x1="64.44" y1="4.18" x2="64.44" y2="4.05" width="1.016" layer="16"/>
-<wire x1="64.33" y1="11.878" x2="54.61" y2="11.878" width="1.016" layer="16"/>
+<wire x1="64.33" y1="11.878" x2="57.15" y2="11.878" width="1.016" layer="16"/>
 <via x="27.94" y="16.51" extent="1-16" drill="0.85" shape="octagon"/>
 <via x="49.53" y="16.51" extent="1-16" drill="0.85" shape="octagon"/>
-<wire x1="54.162" y1="11.878" x2="54.61" y2="11.878" width="1.016" layer="16"/>
+<wire x1="57.15" y1="11.878" x2="54.61" y2="11.878" width="1.016" layer="16"/>
 <wire x1="54.61" y1="11.878" x2="54.162" y2="11.878" width="1.016" layer="16"/>
 <wire x1="54.162" y1="11.878" x2="49.53" y2="16.51" width="1.016" layer="16"/>
 <wire x1="25.4" y1="16.51" x2="27.94" y2="16.51" width="1.016" layer="16"/>
 <wire x1="27.94" y1="16.51" x2="49.53" y2="16.51" width="1.016" layer="1"/>
+<contactref element="JP8" pad="1"/>
+<wire x1="57.15" y1="8.89" x2="57.15" y2="11.878" width="0.8128" layer="16"/>
 </signal>
 <signal name="N$2">

Commit message: Update
Parts:
- renumbered IC1 to U3, IC2 to U2, U$1 to U1
Changed lines of the file:
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@@
 </autorouter>
 <elements>
-<element name="IC1" library="uln-udn" library_urn="urn:adsk.eagle:library:407" package="DIL16" package3d_urn="urn:adsk.eagle:package:30239/1" value="ULN2003AN" x="69.76" y="40.84" rot="R270"/>
-<element name="IC2" library="v-reg" library_urn="urn:adsk.eagle:library:409" package="78XXS" package3d_urn="urn:adsk.eagle:package:30342/1" value="" x="74.42" y="11.78" rot="R270"/>
+<element name="U3" library="uln-udn" library_urn="urn:adsk.eagle:library:407" package="DIL16" package3d_urn="urn:adsk.eagle:package:30239/1" value="ULN2003AN" x="69.76" y="40.84" rot="R270"/>
+<element name="U2" library="v-reg" library_urn="urn:adsk.eagle:library:409" package="78XXS" package3d_urn="urn:adsk.eagle:package:30342/1" value="" x="74.42" y="11.78" rot="R270"/>
 <element name="X1" library="con-ptr500" library_urn="urn:adsk.eagle:library:181" package="AK300/2" package3d_urn="urn:adsk.eagle:package:9881/1" value="" x="82.6" y="13.05" rot="R90">
 <attribute name="MF" value="" x="82.6" y="13.05" size="1.778" layer="27" rot="R90" display="off"/>
@@
 <attribute name="SPICEPREFIX" value="C" x="63.17" y="4.05" size="1.778" layer="27" rot="R180" display="off"/>
 </element>
-<element name="U$1" library="Lolin" package="LOLIN" value="" x="39.37" y="33.02" rot="R270"/>
+<element name="U1" library="Lolin" package="LOLIN" value="" x="39.37" y="33.02" rot="R270"/>
 <element name="X2" library="con-ptr500" library_urn="urn:adsk.eagle:library:181" package="AK300/4" package3d_urn="urn:adsk.eagle:package:9879/1" value="" x="82.55" y="45.72" rot="R90">
 <attribute name="MF" value="" x="82.55" y="45.72" size="1.778" layer="27" rot="R90" display="off"/>
@@
 <contactref element="C3" pad="2"/>
 <contactref element="C1" pad="-"/>
-<contactref element="IC2" pad="GND"/>
-<contactref element="IC1" pad="8"/>
+<contactref element="U2" pad="GND"/>
+<contactref element="U3" pad="8"/>
 <contactref element="X1" pad="1"/>
 <polygon width="0.1524" layer="16">
@@
 <vertex x="0" y="54.61"/>
 </polygon>
-<contactref element="U$1" pad="G"/>
-<contactref element="U$1" pad="G1"/>
-<contactref element="U$1" pad="G2"/>
-<contactref element="U$1" pad="G3"/>
-<contactref element="U$1" pad="G4"/>
+<contactref element="U1" pad="G"/>
+<contactref element="U1" pad="G1"/>
+<contactref element="U1" pad="G2"/>
+<contactref element="U1" pad="G3"/>
+<contactref element="U1" pad="G4"/>
 <contactref element="JP7" pad="1"/>
 </signal>
 <signal name="+12V">
-<contactref element="IC2" pad="IN"/>
+<contactref element="U2" pad="IN"/>
 <contactref element="C1" pad="+"/>
 <contactref element="C3" pad="1"/>
 <contactref element="X1" pad="2"/>
-<contactref element="IC1" pad="9"/>
+<contactref element="U3" pad="9"/>
 <wire x1="82.6" y1="15.5392" x2="81.3808" y2="14.32" width="1.016" layer="16"/>
 <wire x1="81.3808" y1="14.32" x2="71.88" y2="14.32" width="1.016" layer="16"/>
@@
 </signal>
 <signal name="+5V">
-<contactref element="IC2" pad="OUT"/>
+<contactref element="U2" pad="OUT"/>
 <contactref element="C4" pad="1"/>
 <contactref element="C2" pad="+"/>
-<contactref element="U$1" pad="VIN"/>
+<contactref element="U1" pad="VIN"/>
 <wire x1="71.88" y1="9.24" x2="69.5" y2="9.24" width="1.016" layer="16"/>
 <wire x1="66.862" y1="11.878" x2="64.33" y2="11.878" width="1.016" layer="16"/>
@@
 </signal>
 <signal name="N$2">
-<contactref element="IC1" pad="16"/>
+<contactref element="U3" pad="16"/>
 <contactref element="X2" pad="4"/>
 <wire x1="73.57" y1="49.73" x2="77.053" y2="53.213" width="1.016" layer="16"/>
@@
 </signal>
 <signal name="N$3">
-<contactref element="IC1" pad="15"/>
+<contactref element="U3" pad="15"/>
 <contactref element="X2" pad="3"/>
 <wire x1="73.57" y1="47.19" x2="76.4" y2="47.19" width="1.016" layer="16"/>
@@
 </signal>
 <signal name="N$4">
-<contactref element="IC1" pad="14"/>
+<contactref element="U3" pad="14"/>
 <contactref element="X2" pad="2"/>
 <wire x1="73.57" y1="44.65" x2="77.27" y2="44.65" width="1.016" layer="16"/>
@@
 </signal>
 <signal name="N$5">
-<contactref element="IC1" pad="13"/>
+<contactref element="U3" pad="13"/>
 <contactref element="X2" pad="1"/>
 <wire x1="82.55" y1="38.227" x2="82.423" y2="38.227" width="1.016" layer="16"/>
@@
 </signal>
 <signal name="N$1">
-<contactref element="U$1" pad="D0"/>
+<contactref element="U1" pad="D0"/>
 <wire x1="21.59" y1="54.61" x2="27.94" y2="54.61" width="1.016" layer="16"/>
 <wire x1="16.51" y1="49.53" x2="16.51" y2="41.91" width="1.016" layer="16"/>
@@
 </signal>
 <signal name="N$9">
-<contactref element="IC1" pad="1"/>
-<contactref element="U$1" pad="D1"/>
+<contactref element="U3" pad="1"/>
+<contactref element="U1" pad="D1"/>
 <contactref element="JP1" pad="1"/>
 <wire x1="53.34" y1="49.53" x2="59.69" y2="49.53" width="0.8128" layer="16"/>
@@
 </signal>
 <signal name="N$10">
-<contactref element="IC1" pad="2"/>
-<contactref element="U$1" pad="D2"/>
+<contactref element="U3" pad="2"/>
+<contactref element="U1" pad="D2"/>
 <contactref element="JP2" pad="1"/>
 <wire x1="53.34" y1="46.99" x2="59.69" y2="46.99" width="0.8128" layer="16"/>
@@
 </signal>
 <signal name="N$11">
-<contactref element="IC1" pad="3"/>
-<contactref element="U$1" pad="D3"/>
+<contactref element="U3" pad="3"/>
+<contactref element="U1" pad="D3"/>
 <contactref element="JP3" pad="1"/>
 <wire x1="53.34" y1="44.45" x2="59.69" y2="44.45" width="0.8128" layer="16"/>
@@
 </signal>
 <signal name="N$12">
-<contactref element="IC1" pad="4"/>
-<contactref element="U$1" pad="D4"/>
+<contactref element="U3" pad="4"/>
+<contactref element="U1" pad="D4"/>
 <contactref element="JP4" pad="1"/>
 <wire x1="53.34" y1="41.91" x2="59.69" y2="41.91" width="0.8128" layer="16"/>
@@
 </signal>
 <signal name="N$16">
-<contactref element="U$1" pad="A0"/>
+<contactref element="U1" pad="A0"/>
 <wire x1="25.4" y1="52.07" x2="22.86" y2="52.07" width="1.016" layer="16"/>
 <wire x1="22.86" y1="52.07" x2="19.05" y2="48.26" width="1.016" layer="16"/>
@@
 <signal name="N$6">
 <contactref element="X3" pad="6"/>
-<contactref element="U$1" pad="D8"/>
+<contactref element="U1" pad="D8"/>
 <wire x1="20.3349375" y1="6.604" x2="43.1650625" y2="6.604" width="1.016" layer="16"/>
 <wire x1="43.1650625" y1="6.604" x2="46.736" y2="10.1749375" width="1.016" layer="16"/>
@@
 </signal>
 <signal name="N$7">
-<contactref element="U$1" pad="D7"/>
+<contactref element="U1" pad="D7"/>
 <contactref element="X3" pad="5"/>
 <wire x1="6.35" y1="16.6116" x2="16.4084" y2="16.6116" width="1.016" layer="16"/>
@@
 <signal name="N$8">
 <contactref element="X3" pad="4"/>
-<contactref element="U$1" pad="D6"/>
+<contactref element="U1" pad="D6"/>
 <wire x1="6.35" y1="21.6154" x2="16.4846" y2="21.6154" width="1.016" layer="16"/>
 <wire x1="19.558" y1="13.1283125" x2="22.0183125" y2="10.668" width="1.016" layer="16"/>
@@
 </signal>
 <signal name="N$13">
-<contactref element="U$1" pad="D5"/>
+<contactref element="U1" pad="D5"/>
 <contactref element="X3" pad="3"/>
 <wire x1="43.18" y1="34.29" x2="35.56" y2="26.67" width="1.016" layer="16"/>
@@
 <signal name="N$14">
 <contactref element="JP5" pad="1"/>
-<contactref element="U$1" pad="RX"/>
+<contactref element="U1" pad="RX"/>
 <wire x1="53.34" y1="24.13" x2="57.15" y2="24.13" width="0.8128" layer="16"/>
 </signal>
 <signal name="N$15">
-<contactref element="U$1" pad="TX"/>
+<contactref element="U1" pad="TX"/>
 <contactref element="JP6" pad="1"/>
 <wire x1="53.34" y1="21.59" x2="57.15" y2="21.59" width="0.8128" layer="16"/>
 </signal>
 <signal name="N$17">
-<contactref element="U$1" pad="3V2"/>
+<contactref element="U1" pad="3V2"/>
 <contactref element="X4" pad="2"/>
 <contactref element="X4" pad="1"/>
