File: Boards/main_plate.sch (EAGLE design)
At the start: 18 parts, among them IC1 ULN2003AN

Commit message: add nodeMCU code
Parts:
- added JP8: (no value), pinhead:PINHD-1X1
Connections:
- net +5V: now also JP8.1
Changed lines of the file:
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@@
 <part name="JP7" library="pinhead" library_urn="urn:adsk.eagle:library:325" deviceset="PINHD-1X1" device="" package3d_urn="urn:adsk.eagle:package:22485/2"/>
 <part name="X4" library="con-ptr500" library_urn="urn:adsk.eagle:library:181" deviceset="AK300/2" device="" package3d_urn="urn:adsk.eagle:package:9881/1"/>
+<part name="JP8" library="pinhead" library_urn="urn:adsk.eagle:library:325" deviceset="PINHD-1X1" device="" package3d_urn="urn:adsk.eagle:package:22485/2"/>
 </parts>
 <sheets>
@@
 <instance part="X4" gate="-1" x="20.32" y="50.8"/>
 <instance part="X4" gate="-2" x="20.32" y="45.72"/>
+<instance part="JP8" gate="G$1" x="55.88" y="20.32" rot="R180"/>
 </instances>
 <busses>
@@
 <wire x1="48.26" y1="20.32" x2="48.26" y2="25.4" width="0.1524" layer="91"/>
 <junction x="48.26" y="20.32"/>
+<pinref part="JP8" gate="G$1" pin="1"/>
+<wire x1="58.42" y1="20.32" x2="48.26" y2="20.32" width="0.1524" layer="91"/>
 </segment>
 <segment>

Commit message: Update
Parts:
- renumbered IC1 to U3, IC2 to U2, U$1 to U1
